File: PCB/MonitorMainPCB/backup/MainBoard.sch (EAGLE design)
At the start: 140 parts, among them IC1 ADS1293, IC2 LP3878MR-ADJ_NOPB, J1 POWER_JACK, J2 USB_B_PTH, J6 2X6 FEMALE, U2 TPS7A4901DGNR, U3 AFE4400_RHA_40, U4 MSP430F149IPAG, Y1 4.096MHz, Y2 8MHz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

Commit message: finishing Main PCB
Parts:
- added C43: 10uF, SparkFun-Retired:10UF-TANT
- added U$6: XJTULOGO, xjtulogo:XJTULOGO
Connections:
- net N$88 renamed STATE
- removed net N$83: J7.6
- removed net N$84: J7.5
- removed net N$85: J7.4
- removed net N$86: J7.3
- removed net N$87: J7.2
- new net EN_BT: J7.6, U4.P2.1/TAINCLK
- net +5V: now also C43.+, J7.5
- net GND: now also C43.-, J7.4
- net URXD0: now also J7.3
- net UTXD0: now also J7.2
