File: PCB/MonitorMainPCB/MainBoard.brd (EAGLE design)
At the start: 94.1 x 100 mm, 130 parts, among them IC1 ADS1293, IC2 LP3878MR-ADJ_NOPB, J1 POWER_JACK, J2 USB_B_PTH, J6 2X6 FEMALE, U2 TPS7A4901DGNR, U3 AFE4400_RHA_40, U4 MSP430F149IPAG, Y1 4.096MHz, Y2 8MHz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

Commit message: finishing Main PCB
Parts:
- added C43: 10uF, SparkFun-Retired:EIA3216
- added D5, D6, D7, D8, D9: RED, SparkFun-LED:LED-0603
- added J7: (no value), SparkFun-Connectors:1X06
- added R47, R48, R49: 10, SparkFun-Resistors:0603
- added R50, R51, R52, R53, R54: 1k, SparkFun-Resistors:0603
- added U$6: XJTULOGO, xjtulogo:XJTULOGO
Connections:
- removed net P11: J6.6
- new net EN_BT: J7.6, U4.21
- new net N$73: D5.C, U4.23
- new net N$74: D6.C, U4.24
- new net N$75: D7.C, U4.25
- new net N$76: D8.C, U4.26
- new net N$77: D9.C, U4.27
- new net N$78: D5.A, R50.2
- new net N$79: D6.A, R51.2
- new net N$80: D7.A, R52.2
- new net N$81: D8.A, R53.2
- new net N$82: D9.A, R54.2
- new net STATE: J7.1
- net +3V3: now also R50.1, R51.1, R52.1, R53.1, R54.1
- net +5V: now also C43.A, J7.5
- net ADC_RDY: now also U4.38
- net AFE_PDN: now also U4.36
- net ALARMB: now also U4.40
- net DIAG_END: now also U4.39
- net DRDYB: now also U4.42
- net GND: now also C43.C, J7.4
- net LED_ALM: now also U4.41
- net MISO: now also R48.2; no longer U4.30
- net MOSI: now also R47.2
- net N$66: now also R47.1, U4.45; no longer U4.20
- net N$71: now also R48.1, U4.46; no longer U4.29
- net N$72: now also R49.1, U4.47; no longer U4.31
- net PD_ALM: now also U4.37
- net SCLK: now also R49.2
- net SS: now also U4.12
- net STE: now also J6.6, U4.13
- net URXD0: now also J7.3
- net UTXD0: now also J7.2
- net XIN_MSP: now also U4.20; no longer U4.13
Routing:
- net ALARMB: track 19.4 -> 219.7 mm, vias 0 -> 6
- net SS: track 19.6 -> 189.9 mm, vias 0 -> 7
- net DRDYB: track 16.4 -> 185.6 mm, vias 0 -> 5
- net DIAG_END: track 11.2 -> 91.0 mm, vias 0 -> 4
- net ADC_RDY: track 9.10 -> 82.3 mm, vias 0 -> 2
- net PD_ALM: track 9.24 -> 80.9 mm, vias 1 -> 3
- net +3V3: track 196.5 -> 263.5 mm, vias 9 -> 11
- net URXD0: track 0.00 -> 66.2 mm, vias 0 -> 1
- net LED_ALM: track 12.4 -> 74.5 mm, vias 0 -> 2
- net GND: track 782.7 -> 842.9 mm, vias 18 -> 19
- net MOSI: track 55.1 -> 112.2 mm, vias 1 -> 4
- net SCLK: track 53.0 -> 109.9 mm, vias 1 -> 5
- net MISO: track 47.0 -> 101.4 mm, vias 1 -> 4
- net UTXD0: track 0.00 -> 54.3 mm, vias 0 -> 1
- net AFE_PDN: track 12.2 -> 66.2 mm, vias 0 -> 2
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Other:
- board text added: "BT CONN"
- board text added: "ECG-PPG Measurement"
- board text added: "Main PCB"
- board text removed: "ECG-PPG Measurement Main PCB"

Commit message: main PCB finished
Parts:
- added U$7: (no value), xjtulogo:MICELOGO
- C13, C17, C18, C19, C20, C22, C23, C24, C43: device SparkFun-Retired:EIA3216 -> SparkFun-Capacitors:1206
- moved U$6 38.9 mm to (79.6, 76.8)
- moved C13 10.2 mm to (48.5, 10.2), turned to 270 degrees
- moved C17 9.77 mm to (52.6, 19.6), turned to 0 degrees
- moved C43 1.71 mm to (84.6, 44.7), turned to 0 degrees
- moved C18 1.61 mm to (72.1, 11.4), turned to 270 degrees
- moved C22 1.53 mm to (67.8, 28.7), turned to 270 degrees
- moved C24 1.20 mm to (78.0, 29.2), turned to 0 degrees
- moved C20 0.49 mm to (82.3, 11.2), turned to 0 degrees
- moved C23 0.20 mm to (77.0, 23.9), turned to 0 degrees
- moved C19 0.13 mm to (82.0, 15.2), turned to 0 degrees
Connections:
- net +5V: now also C43.1; no longer C43.A
- net GND: now also C13.2, C17.2, C18.2, C19.2, C20.2, C22.2, C23.2, C24.2, C43.2; no longer C13.C, C17.C, C18.C, C19.C, C20.C, C22.C, C23.C, C24.C, C43.C
- net N$18: now also C18.1; no longer C18.A
- net N$23: now also C19.1; no longer C19.A
- net N$24: now also C20.1; no longer C20.A
- net N$25: now also C17.1; no longer C13.A
- net N$28: now also C23.1; no longer C23.A
- net N$29: now also C13.1; no longer C17.A
- net N$30: now also C24.1; no longer C24.A
- net RX_SUP: now also C22.1; no longer C22.A
Routing:
- net GND: track 842.9 -> 845.2 mm
- net +5V: track 216.3 -> 217.9 mm
- net N$18: track 11.1 -> 12.4 mm
- added copper zone on layer 16, net GND
Other:
- board text added: "BSL"
- board text added: "EN"
- board text added: "HUMSTER TEAM, XJTU-BME"
- board text added: "MCU MODULE"
- board text added: "NC"
- board text added: "PCB by Jingjie Li"
- board text added: "RESET BOTTOMS"
- board text added: "RST_MSP"
- board text added: "RX"
- board text added: "TX"
- board text added: "U3"
- board text added: "U5"
- board text added: "UART"
- board text removed: "By Jingjie Li, XJTU-BME"
