File: PCB/MonitorMainPCB/MainBoard.brd (EAGLE design)
At the start: 94.1 x 100 mm, 148 parts, among them IC1 ADS1293, IC2 LP3878MR-ADJ_NOPB, J1 POWER_JACK, J2 USB_B_PTH, J6 2X6 FEMALE, U2 TPS7A4901DGNR, U3 AFE4400_RHA_40, U4 MSP430F149IPAG, Y1 4.096MHz, Y2 8MHz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

Commit message: restart
Parts:
- moved C7 1.51 mm to (20.3, 58.2), flipped to the top
- flipped C10 to the top, turned to 180 degrees
- flipped C11 to the top, turned to 0 degrees
- flipped C5 to the top
- flipped C6 to the top
- flipped R2 to the top, turned to 0 degrees
Routing:
- net GND: track 870.5 -> 877.3 mm, vias 21 -> 26
- net N$1: track 7.81 -> 12.0 mm, vias 1 -> 2
- net +3V3: track 263.5 -> 266.4 mm, vias 11 -> 9
- net RLDIN: track 33.4 -> 31.1 mm
- net N$10: track 6.88 -> 6.76 mm, vias 2 -> 0
