File: PCB/MonitorMainPCB/MainBoard.sch (EAGLE design)
At the start: 126 parts, among them IC1 ADS1293, IC2 LP3878MR-ADJ_NOPB, J1 POWER_JACK, J2 USB_B_PTH, J6 2X6 FEMALE, U2 TPS7A4901DGNR, U3 AFE4400_RHA_40, U4 MSP430F149IPAG, Y1 4.096MHz, Y2 8MHz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

Commit message: finishing Main PCB
Parts:
- added C43: 10uF, SparkFun-Retired:10UF-TANT
- added D5, D6, D7, D8, D9: RED, SparkFun-LED:LED-RED0603
- added J7: (no value), SparkFun-Connectors:CONN_06SILK_FEMALE_PTH
- added R47, R48, R49: 10, SparkFun-Resistors:10OHM-0603-1/10W-1%
- added R50, R51, R52, R53, R54: 1k, SparkFun-Resistors:1KOHM-0603-1/10W-1%
- added U$6: XJTULOGO, xjtulogo:XJTULOGO
Connections:
- removed net P11: J6.6
- new net EN_BT: J7.6, U4.P2.1/TAINCLK
- new net N$73: D5.C, U4.P2.3/CA0/TA1
- new net N$74: D6.C, U4.P2.4/CA1/TA2
- new net N$75: D7.C, U4.P2.5/ROSC
- new net N$76: D8.C, U4.P2.6/ADC12CLK
- new net N$77: D9.C, U4.P2.7/TA0
- new net N$78: D5.A, R50.2
- new net N$79: D6.A, R51.2
- new net N$80: D7.A, R52.2
- new net N$81: D8.A, R53.2
- new net N$82: D9.A, R54.2
- new net STATE: J7.1
- net +3V3: now also R50.1, R51.1, R52.1, R53.1, R54.1
- net +5V: now also C43.+, J7.5
- net ADC_RDY: now also U4.P4.2/TB2
- net AFE_PDN: now also U4.P4.0/TB0
- net ALARMB: now also U4.P4.4/TB4
- net DIAG_END: now also U4.P4.3/TB3
- net DRDYB: now also U4.P4.6/TB6
- net GND: now also C43.-, J7.4
- net LED_ALM: now also U4.P4.5/TB5
- net MISO: now also R48.2; no longer U4.P3.2/SOMI0
- net MOSI: now also R47.2
- net N$66: now also R47.1, U4.P5.1/SIMO1; no longer U4.P2.0/ACLK
- net N$71: now also R48.1, U4.P5.2/SOMI1; no longer U4.P3.1/SIMO0
- net N$72: now also R49.1, U4.P5.3/UCLK1; no longer U4.P3.3/UCLK0
- net PD_ALM: now also U4.P4.1/TB1
- net SCLK: now also R49.2
- net SS: now also U4.P1.0/TACLK
- net STE: now also J6.6, U4.P1.1/TA0
- net URXD0: now also J7.3
- net UTXD0: now also J7.2
- net XIN_MSP: now also U4.P2.0/ACLK; no longer U4.P1.1/TA0

Commit message: main PCB finished
Parts:
- C13, C17, C18, C19, C20, C22, C23, C24, C43: device SparkFun-Retired:10UF-TANT -> SparkFun-Capacitors:10UF-1206-6.3V-20%
Connections:
- net +5V: now also C43.1; no longer C43.+
- net GND: now also C13.2, C17.2, C18.2, C19.2, C20.2, C22.2, C23.2, C24.2, C43.2; no longer C13.-, C17.-, C18.-, C19.-, C20.-, C22.-, C23.-, C24.-, C43.-
- net N$18: now also C18.1; no longer C18.+
- net N$23: now also C19.1; no longer C19.+
- net N$24: now also C20.1; no longer C20.+
- net N$25: now also C17.1; no longer C13.+
- net N$28: now also C23.1; no longer C23.+
- net N$29: now also C13.1; no longer C17.+
- net N$30: now also C24.1; no longer C24.+
- net RX_SUP: now also C22.1; no longer C22.+
